File: kicad/fourkey/fourkey.sch (KiCad schematic (older format))
At the start: 5 parts, among them U1 TEENSY2.0

Commit message: Mostly fourkey PCB work
Parts:
- removed U1: TEENSY2.0, footprint:TEENSY_2.0, symbol TEENSY2.0
- added D1, D2, D3, D4: LED, LEDs:LED-3MM, symbol LED
- added P1: CONN_01X06, Pin_Headers:Pin_Header_Straight_1x06, symbol CONN_01X06
- added R1: RESISTOR, footprint:RESISTOR, symbol RESISTOR
Connections:
- net COL0: now also P1.1 (P1)
- net COL1: now also P1.2 (P2)
- net GND: now also D1.2 (K), D2.2 (K), D3.2 (K), D4.2 (K), P1.6 (P6)
- net ROW0: now also P1.3 (P3)
- net ROW1: now also P1.4 (P4)
- new net: D1.1 (A), D2.1 (A), D3.1 (A), D4.1 (A), R1.1
- new net LED: P1.5 (P5), R1.2
Changed lines of the file:
@@
 $EndDescr
-$Comp
-L TEENSY2.0 U1
-U 1 1 54F8FFED
-P 1500 2250
-F 0 "U1" V 1550 2250 60  0000 C CNN
-F 1 "TEENSY2.0" V 1450 2250 60  0000 C CNN
-F 2 "footprint:TEENSY_2.0" H 1500 2250 60  0001 C CNN
-F 3 "" H 1500 2250 60  0000 C CNN
-	1    1500 2250
-	1    0    0    -1
-$EndComp
 $Comp
 L SWITCH_DIODE 0;0
@@
 F 3 "" H 4200 2200 60  0000 C CNN
 	1    4200 2200
+	1    0    0    -1
+$EndComp
+Text Label 2700 1300 0    60   ~ 0
+COL0
+Text Label 3700 1300 0    60   ~ 0
+COL1
+Text Label 2500 1800 0    60   ~ 0
+ROW0
+Text Label 2500 2500 0    60   ~ 0
+ROW1
+Text Label 1950 1650 0    60   ~ 0
+COL0
+Text Label 1950 1750 0    60   ~ 0
+COL1
+Text Label 1950 1850 0    60   ~ 0
+ROW0
+Text Label 1950 1950 0    60   ~ 0
+ROW1
+$Comp
+L CONN_01X06 P1
+U 1 1 54FA251A
+P 1750 1900
+F 0 "P1" H 1750 2250 50  0000 C CNN
+F 1 "CONN_01X06" V 1850 1900 50  0000 C CNN
+F 2 "Pin_Headers:Pin_Header_Straight_1x06" H 1750 1900 60  0001 C CNN
+F 3 "" H 1750 1900 60  0000 C CNN
+	1    1750 1900
+	-1   0    0    -1
+$EndComp
+Text Label 1950 2050 0    60   ~ 0
+LED
+Text Label 1950 2150 0    60   ~ 0
+GND
+$Comp
+L LED D1
+U 1 1 54FA26EC
+P 5700 1400
+F 0 "D1" H 5700 1500 50  0000 C CNN
+F 1 "LED" H 5700 1300 50  0000 C CNN
+F 2 "LEDs:LED-3MM" H 5700 1400 60  0001 C CNN
+F 3 "" H 5700 1400 60  0000 C CNN
+	1    5700 1400
+	1    0    0    -1
+$EndComp
+$Comp
+L LED D2
+U 1 1 54FA2752
+P 5700 1700
+F 0 "D2" H 5700 1800 50  0000 C CNN
+F 1 "LED" H 5700 1600 50  0000 C CNN
+F 2 "LEDs:LED-3MM" H 5700 1700 60  0001 C CNN
+F 3 "" H 5700 1700 60  0000 C CNN
+	1    5700 1700
+	1    0    0    -1
+$EndComp
+$Comp
+L LED D3
+U 1 1 54FA2775
+P 5700 2000
+F 0 "D3" H 5700 2100 50  0000 C CNN
+F 1 "LED" H 5700 1900 50  0000 C CNN
+F 2 "LEDs:LED-3MM" H 5700 2000 60  0001 C CNN
+F 3 "" H 5700 2000 60  0000 C CNN
+	1    5700 2000
+	1    0    0    -1
+$EndComp
+$Comp
+L LED D4
+U 1 1 54FA279C
+P 5700 2300
+F 0 "D4" H 5700 2400 50  0000 C CNN
+F 1 "LED" H 5700 2200 50  0000 C CNN
+F 2 "LEDs:LED-3MM" H 5700 2300 60  0001 C CNN
+F 3 "" H 5700 2300 60  0000 C CNN
+	1    5700 2300
 	1    0    0    -1
 $EndComp
@@
 	3000 2500 3000 2300
 Connection ~ 3000 2500
-Text Label 2700 1300 0    60   ~ 0
-COL0
-Text Label 3700 1300 0    60   ~ 0
-COL1
-Text Label 2500 1800 0    60   ~ 0
-ROW0
-Text Label 2500 2500 0    60   ~ 0
-ROW1
 Wire Wire Line
-	2100 950  2200 950
+	5500 1400 5500 2300
+Connection ~ 5500 1700
+Connection ~ 5500 2000
 Wire Wire Line
-	2100 1050 2200 1050
+	5500 1400 5300 1400
+Text Label 4800 1400 2    60   ~ 0
+LED
 Wire Wire Line
-	2100 1150 2200 1150
+	5900 1400 5900 2300
+Connection ~ 5900 1700
+Connection ~ 5900 2000
 Wire Wire Line
-	2100 1250 2200 1250
-Text Label 2200 950  0    60   ~ 0
-COL0
-Text Label 2200 1050 0    60   ~ 0
-COL1
-Text Label 2200 1150 0    60   ~ 0
-ROW0
-Text Label 2200 1250 0    60   ~ 0
-ROW1
+	5900 2300 6100 2300
+Text Label 6100 2300 0    60   ~ 0
+GND
+$Comp
+L RESISTOR R1
+U 1 1 54FA2AE0
+P 5050 1400
+F 0 "R1" V 5050 1300 50  0000 C CNN
+F 1 "RESISTOR" V 5050 1500 50  0000 C CNN
+F 2 "footprint:RESISTOR" H 5050 1400 60  0001 C CNN
+F 3 "" H 5050 1400 60  0000 C CNN
+	1    5050 1400
+	0    1    1    0
+$EndComp
 $EndSCHEMATC

Commit message: More FourKey work, including Gerber files
Parts:
- removed D1, D2, D3, D4: LED, LEDs:LED-3MM, symbol LED
- removed P1: CONN_01X06, Pin_Headers:Pin_Header_Straight_1x06, symbol CONN_01X06
- removed R1: RESISTOR, footprint:RESISTOR, symbol RESISTOR
- added J1: 4PIN, Pin_Headers:Pin_Header_Straight_1x04, symbol 4PIN
Connections:
- net COL0: now also J1.1
- net COL1: now also J1.2
- net ROW0: now also J1.3
- net ROW1: now also J1.4
Changed lines of the file:
@@
 Text Label 1950 1950 0    60   ~ 0
 ROW1
-$Comp
-L CONN_01X06 P1
-U 1 1 54FA251A
-P 1750 1900
-F 0 "P1" H 1750 2250 50  0000 C CNN
-F 1 "CONN_01X06" V 1850 1900 50  0000 C CNN
-F 2 "Pin_Headers:Pin_Header_Straight_1x06" H 1750 1900 60  0001 C CNN
-F 3 "" H 1750 1900 60  0000 C CNN
-	1    1750 1900
-	-1   0    0    -1
-$EndComp
-Text Label 1950 2050 0    60   ~ 0
-LED
-Text Label 1950 2150 0    60   ~ 0
-GND
-$Comp
-L LED D1
-U 1 1 54FA26EC
-P 5700 1400
-F 0 "D1" H 5700 1500 50  0000 C CNN
-F 1 "LED" H 5700 1300 50  0000 C CNN
-F 2 "LEDs:LED-3MM" H 5700 1400 60  0001 C CNN
-F 3 "" H 5700 1400 60  0000 C CNN
-	1    5700 1400
-	1    0    0    -1
-$EndComp
-$Comp
-L LED D2
-U 1 1 54FA2752
-P 5700 1700
-F 0 "D2" H 5700 1800 50  0000 C CNN
-F 1 "LED" H 5700 1600 50  0000 C CNN
-F 2 "LEDs:LED-3MM" H 5700 1700 60  0001 C CNN
-F 3 "" H 5700 1700 60  0000 C CNN
-	1    5700 1700
-	1    0    0    -1
-$EndComp
-$Comp
-L LED D3
-U 1 1 54FA2775
-P 5700 2000
-F 0 "D3" H 5700 2100 50  0000 C CNN
-F 1 "LED" H 5700 1900 50  0000 C CNN
-F 2 "LEDs:LED-3MM" H 5700 2000 60  0001 C CNN
-F 3 "" H 5700 2000 60  0000 C CNN
-	1    5700 2000
-	1    0    0    -1
-$EndComp
-$Comp
-L LED D4
-U 1 1 54FA279C
-P 5700 2300
-F 0 "D4" H 5700 2400 50  0000 C CNN
-F 1 "LED" H 5700 2200 50  0000 C CNN
-F 2 "LEDs:LED-3MM" H 5700 2300 60  0001 C CNN
-F 3 "" H 5700 2300 60  0000 C CNN
-	1    5700 2300
-	1    0    0    -1
-$EndComp
 Wire Wire Line
 	2700 1300 2700 2200
@@
 	3000 2500 3000 2300
 Connection ~ 3000 2500
-Wire Wire Line
-	5500 1400 5500 2300
-Connection ~ 5500 1700
-Connection ~ 5500 2000
-Wire Wire Line
-	5500 1400 5300 1400
-Text Label 4800 1400 2    60   ~ 0
-LED
-Wire Wire Line
-	5900 1400 5900 2300
-Connection ~ 5900 1700
-Connection ~ 5900 2000
-Wire Wire Line
-	5900 2300 6100 2300
-Text Label 6100 2300 0    60   ~ 0
-GND
 $Comp
-L RESISTOR R1
-U 1 1 54FA2AE0
-P 5050 1400
-F 0 "R1" V 5050 1300 50  0000 C CNN
-F 1 "RESISTOR" V 5050 1500 50  0000 C CNN
-F 2 "footprint:RESISTOR" H 5050 1400 60  0001 C CNN
-F 3 "" H 5050 1400 60  0000 C CNN
-	1    5050 1400
-	0    1    1    0
+L 4PIN J1
+U 1 1 54FC9E1C
+P 1750 1800
+F 0 "J1" H 1700 2050 60  0000 C CNN
+F 1 "4PIN" H 1700 1550 60  0000 C CNN
+F 2 "Pin_Headers:Pin_Header_Straight_1x04" H 1750 1800 60  0001 C CNN
+F 3 "" H 1750 1800 60  0000 C CNN
+	1    1750 1800
+	1    0    0    -1
 $EndComp
 $EndSCHEMATC
